Commit message: feat: use main.sdf world, model is attached to groung plane

File: 05_ros2_control/panda_gz_ros2_ctrl/panda_description/urdf/panda.urdf.xacro (robot description, xacro)
@@ -1,8 +1,10 @@
 <?xml version="1.0" ?>
-<!-- =================================================================================== -->
-<!-- |    This document was autogenerated by xacro from /opt/ros/kinetic/share/moveit_resources/panda_description/urdf/panda.urdf | -->
-<!-- |    EDITING THIS FILE BY HAND IS NOT RECOMMENDED                                 | -->
-<!-- =================================================================================== -->
-<robot name="panda" xmlns:xacro="http://www.ros.org/wiki/xacro">
+<robot name="panda"
+    xmlns:xacro="http://www.ros.org/wiki/xacro">
+    <link name="world"/>
+    <joint name="fixed" type="fixed">
+        <parent link="world"/>
+        <child link="panda_link0"/>
+    </joint>
     <link name="panda_link0">
         <visual>
@@ -17,7 +19,7 @@
         </collision>
         <inertial>
-          <origin xyz="-0.041018 -0.00014 0.049974" rpy="0 0 0" />
-          <mass value="0.629769"/>
-          <inertia ixx="0.00315" iyy="0.00388" izz="0.004285" ixy="8.2904E-7" ixz="0.00015" iyz="8.2299E-6"/>
+            <origin xyz="-0.041018 -0.00014 0.049974" rpy="0 0 0" />
+            <mass value="0.629769"/>
+            <inertia ixx="0.00315" iyy="0.00388" izz="0.004285" ixy="8.2904E-7" ixz="0.00015" iyz="8.2299E-6"/>
         </inertial>
     </link>
@@ -34,7 +36,7 @@
         </collision>
         <inertial>
-          <origin xyz="0.003875 0.002081 -0.04762" rpy="0 0 0" />
-          <mass value="4.970684"/>
-          <inertia ixx="0.70337" iyy="0.70661" izz="0.009117" ixy="-0.000139" ixz="0.006772" iyz="0.019169"/>
+            <origin xyz="0.003875 0.002081 -0.04762" rpy="0 0 0" />
+            <mass value="4.970684"/>
+            <inertia ixx="0.70337" iyy="0.70661" izz="0.009117" ixy="-0.000139" ixz="0.006772" iyz="0.019169"/>
         </inertial>
     </link>
@@ -60,7 +62,7 @@
         </collision>
         <inertial>
-          <origin xyz="-0.003141 -0.02872  0.003495" rpy="0 0 0" />
-          <mass value="0.646926"/>
-          <inertia ixx="0.007962" iyy="2.811E-2" izz="2.5995E-2" ixy="-3.925E-3" ixz="1.0254E-2" iyz="7.04E-4"/>
+            <origin xyz="-0.003141 -0.02872  0.003495" rpy="0 0 0" />
+            <mass value="0.646926"/>
+            <inertia ixx="0.007962" iyy="2.811E-2" izz="2.5995E-2" ixy="-3.925E-3" ixz="1.0254E-2" iyz="7.04E-4"/>
         </inertial>
     </link>
@@ -86,7 +88,7 @@
         </collision>
         <inertial>
-          <origin xyz="2.7518E-2 3.9252E-2 -6.6502E-2" rpy="0 0 0" />
-          <mass value="3.228604"/>
-          <inertia ixx="3.7242E-2" iyy="3.6155E-2" izz="1.083E-2" ixy="-4.761E-3" ixz="-1.1396E-2" iyz="-1.2805E-2"/>
+            <origin xyz="2.7518E-2 3.9252E-2 -6.6502E-2" rpy="0 0 0" />
+            <mass value="3.228604"/>
+            <inertia ixx="3.7242E-2" iyy="3.6155E-2" izz="1.083E-2" ixy="-4.761E-3" ixz="-1.1396E-2" iyz="-1.2805E-2"/>
         </inertial>
     </link>
@@ -112,7 +114,7 @@
         </collision>
         <inertial>
-          <origin xyz="-5.317E-2 1.04419E-1 2.7454E-2" rpy="0 0 0" />
-          <mass value="3.587895"/>
-          <inertia ixx="2.5853E-2" iyy="1.9552E-2" izz="2.8323E-2" ixy="7.796E-3" ixz="-1.332E-3" iyz="8.641E-3"/>
+            <origin xyz="-5.317E-2 1.04419E-1 2.7454E-2" rpy="0 0 0" />
+            <mass value="3.587895"/>
+            <inertia ixx="2.5853E-2" iyy="1.9552E-2" izz="2.8323E-2" ixy="7.796E-3" ixz="-1.332E-3" iyz="8.641E-3"/>
         </inertial>
     </link>
@@ -138,7 +140,7 @@
         </collision>
         <inertial>
-          <origin xyz="-1.1953E-2 4.1065E-2 -3.8437E-2" rpy="0 0 0" />
-          <mass value="1.225946"/>
-          <inertia ixx="3.5549E-2" iyy="2.9474E-2" izz="8.627E-3" ixy="-2.117E-3" ixz="-4.037E-3" iyz="2.29E-4"/>
+            <origin xyz="-1.1953E-2 4.1065E-2 -3.8437E-2" rpy="0 0 0" />
+            <mass value="1.225946"/>
+            <inertia ixx="3.5549E-2" iyy="2.9474E-2" izz="8.627E-3" ixy="-2.117E-3" ixz="-4.037E-3" iyz="2.29E-4"/>
         </inertial>
     </link>
@@ -164,7 +166,7 @@
         </collision>
         <inertial>
-          <origin xyz="6.0149E-2 -1.4117E-2 -1.0517E-2" rpy="0 0 0" />
-          <mass value="1.666555"/>
-          <inertia ixx="1.964E-3" iyy="4.354E-3" izz="5.433E-3" ixy="1.09E-4" ixz="-1.158E-3" iyz="3.41E-4"/>
+            <origin xyz="6.0149E-2 -1.4117E-2 -1.0517E-2" rpy="0 0 0" />
+            <mass value="1.666555"/>
+            <inertia ixx="1.964E-3" iyy="4.354E-3" izz="5.433E-3" ixy="1.09E-4" ixz="-1.158E-3" iyz="3.41E-4"/>
         </inertial>
     </link>
@@ -190,7 +192,7 @@
         </collision>
         <inertial>
-          <origin xyz="1.0517E-2 -4.252E-3 6.1597E-2" rpy="0 0 0" />
-          <mass value="7.35522E-1"/>
-          <inertia ixx="1.2516E-2" iyy="1.0027E-2" izz="4.815E-3" ixy="-4.28E-4" ixz="-1.19E-3" iyz="-7.41E-4"/>
+            <origin xyz="1.0517E-2 -4.252E-3 6.1597E-2" rpy="0 0 0" />
+            <mass value="7.35522E-1"/>
+            <inertia ixx="1.2516E-2" iyy="1.0027E-2" izz="4.815E-3" ixy="-4.28E-4" ixz="-1.19E-3" iyz="-7.41E-4"/>
         </inertial>
     </link>
@@ -228,7 +230,7 @@
         </collision>
         <inertial>
-          <origin xyz="-0.01 0 0.03" rpy="0 0 0" />
-          <mass value="0.73"/>
-          <inertia ixx="0.001" iyy="0.0025" izz="0.0017" ixy="0" ixz="0" iyz="0"/>
+            <origin xyz="-0.01 0 0.03" rpy="0 0 0" />
+            <mass value="0.73"/>
+            <inertia ixx="0.001" iyy="0.0025" izz="0.0017" ixy="0" ixz="0" iyz="0"/>
         </inertial>
     </link>
@@ -245,7 +247,7 @@
         </collision>
         <inertial>
-          <origin xyz="0 0 0" rpy="0 0 0" />
-          <mass value="0.015"/>
-          <inertia ixx="2.375E-6" iyy="2.375E-6" izz="7.5E-7" ixy="0" ixz="0" iyz="0"/>
+            <origin xyz="0 0 0" rpy="0 0 0" />
+            <mass value="0.015"/>
+            <inertia ixx="2.375E-6" iyy="2.375E-6" izz="7.5E-7" ixy="0" ixz="0" iyz="0"/>
         </inertial>
     </link>
@@ -264,7 +266,7 @@
         </collision>
         <inertial>
-          <origin xyz="0 0 0" rpy="0 0 0" />
-          <mass value="0.15"/>
-          <inertia ixx="2.375E-6" iyy="2.375E-6" izz="7.5E-7" ixy="0" ixz="0" iyz="0"/>
+            <origin xyz="0 0 0" rpy="0 0 0" />
+            <mass value="0.15"/>
+            <inertia ixx="2.375E-6" iyy="2.375E-6" izz="7.5E-7" ixy="0" ixz="0" iyz="0"/>
         </inertial>
     </link>

Commit message: feat: add controllers for revolute joints, and set upright initial position for the Panda arm

File: 05_ros2_control/panda_gz_ros2_ctrl/panda_description/urdf/panda.urdf.xacro (robot description, xacro)
@@ -288,3 +288,99 @@
         <dynamics damping="0.3" />
     </joint>
+    <ros2_control name="GazeboSimSystem" type="system">
+        <hardware>
+            <plugin>gz_ros2_control/GazeboSimSystem</plugin>
+        </hardware>
+        <!-- A stable, upright initial position for the Panda arm -->
+        <!-- Joint 1 -->
+        <joint name="panda_joint1">
+            <command_interface name="position">
+                <param name="min">-2.8973</param>
+                <param name="max">2.8973</param>
+            </command_interface>
+            <state_interface name="position">
+                <param name="initial_value">0.0</param>
+            </state_interface>
+            <state_interface name="velocity"/>
+            <state_interface name="effort"/>
+        </joint>
+        <!-- Joint 2 -->
+        <joint name="panda_joint2">
+            <command_interface name="position">
+                <param name="min">-1.7628</param>
+                <param name="max">1.7628</param>
+            </command_interface>
+            <state_interface name="position">
+                <param name="initial_value">-0.785</param> <!-- -45 degrees -->
+            </state_interface>
+            <state_interface name="velocity"/>
+            <state_interface name="effort"/>
+        </joint>
+        <!-- Joint 3 -->
+        <joint name="panda_joint3">
+            <command_interface name="position">
+                <param name="min">-2.8973</param>
+                <param name="max">2.8973</param>
+            </command_interface>
+            <state_interface name="position">
+                <param name="initial_value">0.0</param>
+            </state_interface>
+            <state_interface name="velocity"/>
+            <state_interface name="effort"/>
+        </joint>
+        <!-- Joint 4 -->
+        <joint name="panda_joint4">
+            <command_interface name="position">
+                <param name="min">-3.0718</param>
+                <param name="max">-0.0698</param>
+            </command_interface>
+            <state_interface name="position">
+                <param name="initial_value">-2.356</param> <!-- -135 degrees -->
+            </state_interface>
+            <state_interface name="velocity"/>
+            <state_interface name="effort"/>
+        </joint>
+        <!-- Joint 5 -->
+        <joint name="panda_joint5">
+            <command_interface name="position">
+                <param name="min">-2.8973</param>
+                <param name="max">2.8973</param>
+            </command_interface>
+            <state_interface name="position">
+                <param name="initial_value">0.0</param>
+            </state_interface>
+            <state_interface name="velocity"/>
+            <state_interface name="effort"/>
+        </joint>
+        <!-- Joint 6 -->
+        <joint name="panda_joint6">
+            <command_interface name="position">
+                <param name="min">-0.0175</param>
+                <param name="max">3.7525</param>
+            </command_interface>
+            <state_interface name="position">
+                <param name="initial_value">1.571</param> <!-- 90 degrees -->
+            </state_interface>
+            <state_interface name="velocity"/>
+            <state_interface name="effort"/>
+        </joint>
+        <!-- Joint 7 -->
+        <joint name="panda_joint7">
+            <command_interface name="position">
+                <param name="min">-2.8973</param>
+                <param name="max">2.8973</param>
+            </command_interface>
+            <state_interface name="position">
+                <param name="initial_value">0.785</param> <!-- 45 degrees -->
+            </state_interface>
+            <state_interface name="velocity"/>
+            <state_interface name="effort"/>
+        </joint>
+    </ros2_control>
+    <gazebo>
+        <!-- Joint state publisher -->
+        <plugin filename="gz_ros2_control-system" name="gz_ros2_control::GazeboSimROS2ControlPlugin">
+            <parameters>$(find panda_gz_ros2_ctrl)/config/controller.yaml</parameters>
+        </plugin>
+    </gazebo>
 </robot>

Commit message: feat: add hand controller with fingers, left is mimic

File: 05_ros2_control/panda_gz_ros2_ctrl/panda_description/urdf/panda.urdf.xacro (robot description, xacro)
@@ -312,5 +312,5 @@
             </command_interface>
             <state_interface name="position">
-                <param name="initial_value">-0.785</param> <!-- -45 degrees -->
+                <param name="initial_value">-0.785</param>                <!-- -45 degrees -->
             </state_interface>
             <state_interface name="velocity"/>
@@ -336,5 +336,5 @@
             </command_interface>
             <state_interface name="position">
-                <param name="initial_value">-2.356</param> <!-- -135 degrees -->
+                <param name="initial_value">-2.356</param>                <!-- -135 degrees -->
             </state_interface>
             <state_interface name="velocity"/>
@@ -360,5 +360,5 @@
             </command_interface>
             <state_interface name="position">
-                <param name="initial_value">1.571</param> <!-- 90 degrees -->
+                <param name="initial_value">1.571</param>                <!-- 90 degrees -->
             </state_interface>
             <state_interface name="velocity"/>
@@ -372,5 +372,27 @@
             </command_interface>
             <state_interface name="position">
-                <param name="initial_value">0.785</param> <!-- 45 degrees -->
+                <param name="initial_value">0.785</param>                <!-- 45 degrees -->
+            </state_interface>
+            <state_interface name="velocity"/>
+            <state_interface name="effort"/>
+        </joint>
+        <!-- Actuated Finger Joint -->
+        <joint name="panda_finger_joint1">
+            <command_interface name="position">
+                <param name="min">0.0</param>
+                <param name="max">0.04</param>
+            </command_interface>
+            <state_interface name="position">
+                <param name="initial_value">0.0</param>  <!-- Start with the gripper closed -->
+            </state_interface>
+            <state_interface name="velocity"/>
+            <state_interface name="effort"/>
+        </joint>
+        <!-- Mimic Finger Joint -->
+        <joint name="panda_finger_joint2">
+            <!-- NOTE: No command_interface for the mimic joint! -->
+            <!-- It still needs a state interface for the joint_state_broadcaster. -->
+            <state_interface name="position">
+                <param name="initial_value">0.0</param>
             </state_interface>
             <state_interface name="velocity"/>

Commit message: feat: add demo control node

File: 05_ros2_control/panda_gz_ros2_ctrl/panda_description/urdf/panda.urdf.xacro (robot description, xacro)
@@ -276,5 +276,5 @@
         <origin rpy="0 0 0" xyz="0 0 0.0584" />
         <axis xyz="0 1 0" />
-        <limit effort="20" lower="0.0" upper="0.04" velocity="0.2" />
+        <limit effort="40" lower="0.0" upper="0.04" velocity="0.2" />
         <dynamics damping="0.3" />
     </joint>
@@ -284,5 +284,5 @@
         <origin rpy="0 0 0" xyz="0 0 0.0584" />
         <axis xyz="0 -1 0" />
-        <limit effort="20" lower="0.0" upper="0.04" velocity="0.2" />
+        <limit effort="40" lower="0.0" upper="0.04" velocity="0.2" />
         <mimic joint="panda_finger_joint1" />
         <dynamics damping="0.3" />

Commit message: feat: add demo control node

File: 05_ros2_control/panda_gz_ros2_ctrl/panda_description/urdf/panda.urdf.xacro (robot description, xacro)
@@ -276,5 +276,5 @@
         <origin rpy="0 0 0" xyz="0 0 0.0584" />
         <axis xyz="0 1 0" />
-        <limit effort="40" lower="0.0" upper="0.04" velocity="0.2" />
+        <limit effort="20" lower="0.0" upper="0.04" velocity="0.2" />
         <dynamics damping="0.3" />
     </joint>
@@ -284,5 +284,5 @@
         <origin rpy="0 0 0" xyz="0 0 0.0584" />
         <axis xyz="0 -1 0" />
-        <limit effort="40" lower="0.0" upper="0.04" velocity="0.2" />
+        <limit effort="20" lower="0.0" upper="0.04" velocity="0.2" />
         <mimic joint="panda_finger_joint1" />
         <dynamics damping="0.3" />
