Commit message: fix: udrf - link to current package, get rid of moveit panda descr dead link

File: 05_ros2_control/panda_gz_ros2_ctrl/panda_description/urdf/panda.urdf.xacro (robot description, xacro)
@@ -10,10 +10,10 @@
         <visual>
             <geometry>
-                <mesh filename="file://$(find moveit_resources_panda_description)/meshes/visual/link0.dae" />
-            </geometry>
-        </visual>
-        <collision>
-            <geometry>
-                <mesh filename="file://$(find moveit_resources_panda_description)/meshes/collision/link0.stl" />
+                <mesh filename="file://$(find panda_gz_ros2_ctrl)/panda_description/meshes/visual/link0.dae" />
+            </geometry>
+        </visual>
+        <collision>
+            <geometry>
+                <mesh filename="file://$(find panda_gz_ros2_ctrl)/panda_description/meshes/collision/link0.stl" />
             </geometry>
         </collision>
@@ -27,10 +27,10 @@
         <visual>
             <geometry>
-                <mesh filename="file://$(find moveit_resources_panda_description)/meshes/visual/link1.dae" />
-            </geometry>
-        </visual>
-        <collision>
-            <geometry>
-                <mesh filename="file://$(find moveit_resources_panda_description)/meshes/collision/link1.stl" />
+                <mesh filename="file://$(find panda_gz_ros2_ctrl)/panda_description/meshes/visual/link1.dae" />
+            </geometry>
+        </visual>
+        <collision>
+            <geometry>
+                <mesh filename="file://$(find panda_gz_ros2_ctrl)/panda_description/meshes/collision/link1.stl" />
             </geometry>
         </collision>
@@ -53,10 +53,10 @@
         <visual>
             <geometry>
-                <mesh filename="file://$(find moveit_resources_panda_description)/meshes/visual/link2.dae" />
-            </geometry>
-        </visual>
-        <collision>
-            <geometry>
-                <mesh filename="file://$(find moveit_resources_panda_description)/meshes/collision/link2.stl" />
+                <mesh filename="file://$(find panda_gz_ros2_ctrl)/panda_description/meshes/visual/link2.dae" />
+            </geometry>
+        </visual>
+        <collision>
+            <geometry>
+                <mesh filename="file://$(find panda_gz_ros2_ctrl)/panda_description/meshes/collision/link2.stl" />
             </geometry>
         </collision>
@@ -79,10 +79,10 @@
         <visual>
             <geometry>
-                <mesh filename="file://$(find moveit_resources_panda_description)/meshes/visual/link3.dae" />
-            </geometry>
-        </visual>
-        <collision>
-            <geometry>
-                <mesh filename="file://$(find moveit_resources_panda_description)/meshes/collision/link3.stl" />
+                <mesh filename="file://$(find panda_gz_ros2_ctrl)/panda_description/meshes/visual/link3.dae" />
+            </geometry>
+        </visual>
+        <collision>
+            <geometry>
+                <mesh filename="file://$(find panda_gz_ros2_ctrl)/panda_description/meshes/collision/link3.stl" />
             </geometry>
         </collision>
@@ -105,10 +105,10 @@
         <visual>
             <geometry>
-                <mesh filename="file://$(find moveit_resources_panda_description)/meshes/visual/link4.dae" />
-            </geometry>
-        </visual>
-        <collision>
-            <geometry>
-                <mesh filename="file://$(find moveit_resources_panda_description)/meshes/collision/link4.stl" />
+                <mesh filename="file://$(find panda_gz_ros2_ctrl)/panda_description/meshes/visual/link4.dae" />
+            </geometry>
+        </visual>
+        <collision>
+            <geometry>
+                <mesh filename="file://$(find panda_gz_ros2_ctrl)/panda_description/meshes/collision/link4.stl" />
             </geometry>
         </collision>
@@ -131,10 +131,10 @@
         <visual>
             <geometry>
-                <mesh filename="file://$(find moveit_resources_panda_description)/meshes/visual/link5.dae" />
-            </geometry>
-        </visual>
-        <collision>
-            <geometry>
-                <mesh filename="file://$(find moveit_resources_panda_description)/meshes/collision/link5.stl" />
+                <mesh filename="file://$(find panda_gz_ros2_ctrl)/panda_description/meshes/visual/link5.dae" />
+            </geometry>
+        </visual>
+        <collision>
+            <geometry>
+                <mesh filename="file://$(find panda_gz_ros2_ctrl)/panda_description/meshes/collision/link5.stl" />
             </geometry>
         </collision>
@@ -157,10 +157,10 @@
         <visual>
             <geometry>
-                <mesh filename="file://$(find moveit_resources_panda_description)/meshes/visual/link6.dae" />
-            </geometry>
-        </visual>
-        <collision>
-            <geometry>
-                <mesh filename="file://$(find moveit_resources_panda_description)/meshes/collision/link6.stl" />
+                <mesh filename="file://$(find panda_gz_ros2_ctrl)/panda_description/meshes/visual/link6.dae" />
+            </geometry>
+        </visual>
+        <collision>
+            <geometry>
+                <mesh filename="file://$(find panda_gz_ros2_ctrl)/panda_description/meshes/collision/link6.stl" />
             </geometry>
         </collision>
@@ -183,10 +183,10 @@
         <visual>
             <geometry>
-                <mesh filename="file://$(find moveit_resources_panda_description)/meshes/visual/link7.dae" />
-            </geometry>
-        </visual>
-        <collision>
-            <geometry>
-                <mesh filename="file://$(find moveit_resources_panda_description)/meshes/collision/link7.stl" />
+                <mesh filename="file://$(find panda_gz_ros2_ctrl)/panda_description/meshes/visual/link7.dae" />
+            </geometry>
+        </visual>
+        <collision>
+            <geometry>
+                <mesh filename="file://$(find panda_gz_ros2_ctrl)/panda_description/meshes/collision/link7.stl" />
             </geometry>
         </collision>
@@ -221,10 +221,10 @@
         <visual>
             <geometry>
-                <mesh filename="file://$(find moveit_resources_panda_description)/meshes/visual/hand.dae" />
-            </geometry>
-        </visual>
-        <collision>
-            <geometry>
-                <mesh filename="file://$(find moveit_resources_panda_description)/meshes/collision/hand.stl" />
+                <mesh filename="file://$(find panda_gz_ros2_ctrl)/panda_description/meshes/visual/hand.dae" />
+            </geometry>
+        </visual>
+        <collision>
+            <geometry>
+                <mesh filename="file://$(find panda_gz_ros2_ctrl)/panda_description/meshes/collision/hand.stl" />
             </geometry>
         </collision>
@@ -238,10 +238,10 @@
         <visual>
             <geometry>
-                <mesh filename="file://$(find moveit_resources_panda_description)/meshes/visual/finger.dae" />
-            </geometry>
-        </visual>
-        <collision>
-            <geometry>
-                <mesh filename="file://$(find moveit_resources_panda_description)/meshes/collision/finger.stl" />
+                <mesh filename="file://$(find panda_gz_ros2_ctrl)/panda_description/meshes/visual/finger.dae" />
+            </geometry>
+        </visual>
+        <collision>
+            <geometry>
+                <mesh filename="file://$(find panda_gz_ros2_ctrl)/panda_description/meshes/collision/finger.stl" />
             </geometry>
         </collision>
@@ -256,5 +256,5 @@
             <origin rpy="0 0 3.14159265359" xyz="0 0 0" />
             <geometry>
-                <mesh filename="file://$(find moveit_resources_panda_description)/meshes/visual/finger.dae" />
+                <mesh filename="file://$(find panda_gz_ros2_ctrl)/panda_description/meshes/visual/finger.dae" />
             </geometry>
         </visual>
@@ -262,5 +262,5 @@
             <origin rpy="0 0 3.14159265359" xyz="0 0 0" />
             <geometry>
-                <mesh filename="file://$(find moveit_resources_panda_description)/meshes/collision/finger.stl" />
+                <mesh filename="file://$(find panda_gz_ros2_ctrl)/panda_description/meshes/collision/finger.stl" />
             </geometry>
         </collision>
